Commit message: Stabilize ToolFrame 6.4 mainline benchmark

File: simtoolreal/assets/urdf/parttoolgen_benchmark/screwdriver_insert_socket/deep_socket_075x075x055.urdf (robot description, URDF)
Before this commit: robot parttoolgen_screwdriver_insert_thin_guide_socket, 1 links, 0 joints
Links:
- link thin_guide_socket: geometry collision box size=0.002 0.012 0.055; collision box size=0.002 0.012 0.055

File: simtoolreal/assets/urdf/parttoolgen_benchmark/screwdriver_insert_socket/deep_socket_wide_048x055.urdf (robot description, URDF)
Before this commit: robot parttoolgen_screwdriver_insert_wide_guide_socket, 1 links, 0 joints
Links:
- link wide_guide_socket: geometry collision box size=0.003 0.030 0.055; collision box size=0.003 0.030 0.055
